Commit message: Add files via upload

File: body.urdf (robot description, URDF)
Before this commit: robot robot, 3 links, 2 joints
Links:
- removed link BackLeg
- removed link FrontLeg
- removed link Torso
- added link 0, mass 1; collision box size=0.5370731890796975 0.5370731890796975 0.5370731890796975; visual box size=0.5370731890796975 0.5370731890796975 0.5370731890796975
- added link 1, mass 1; collision box size=0.9539582071715343 0.9539582071715343 0.9539582071715343; visual box size=0.9539582071715343 0.9539582071715343 0.9539582071715343
- added link 2, mass 1; collision box size=0.4389833911819153 0.4389833911819153 0.4389833911819153; visual box size=0.4389833911819153 0.4389833911819153 0.4389833911819153
- added link 3, mass 1; collision box size=0.19592352502965538 0.19592352502965538 0.19592352502965538; visual box size=0.19592352502965538 0.19592352502965538 0.19592352502965538
- added link 4, mass 1; collision box size=0.7692210046700337 0.7692210046700337 0.7692210046700337; visual box size=0.7692210046700337 0.7692210046700337 0.7692210046700337
- added link 5, mass 1; collision box size=0.7142998132910272 0.7142998132910272 0.7142998132910272; visual box size=0.7142998132910272 0.7142998132910272 0.7142998132910272
- added link 6, mass 1; collision box size=0.8098941087802216 0.8098941087802216 0.8098941087802216; visual box size=0.8098941087802216 0.8098941087802216 0.8098941087802216
- added link 7, mass 1; collision box size=0.5697428202496254 0.5697428202496254 0.5697428202496254; visual box size=0.5697428202496254 0.5697428202496254 0.5697428202496254
Joints:
- removed joint BackLeg-Torso
- removed joint FrontLeg-Torso
- added joint 0_1: type revolute, parent 0, child 1, origin xyz=0.26853659453984874 0 0.5 rpy=0 0 0, axis 0 0 1, limit lower=-3.14159 upper=3.14159 effort=0.0 velocity=0.0
- added joint 1_2: type revolute, parent 1, child 2, origin xyz=0.9539582071715343 0 0 rpy=0 0 0, axis 0 0 1, limit lower=-3.14159 upper=3.14159 effort=0.0 velocity=0.0
- added joint 2_3: type revolute, parent 2, child 3, origin xyz=0.4389833911819153 0 0 rpy=0 0 0, axis 0 0 1, limit lower=-3.14159 upper=3.14159 effort=0.0 velocity=0.0
- added joint 3_4: type revolute, parent 3, child 4, origin xyz=0.19592352502965538 0 0 rpy=0 0 0, axis 0 0 1, limit lower=-3.14159 upper=3.14159 effort=0.0 velocity=0.0
- added joint 4_5: type revolute, parent 4, child 5, origin xyz=0.7692210046700337 0 0 rpy=0 0 0, axis 0 0 1, limit lower=-3.14159 upper=3.14159 effort=0.0 velocity=0.0
- added joint 5_6: type revolute, parent 5, child 6, origin xyz=0.7142998132910272 0 0 rpy=0 0 0, axis 0 0 1, limit lower=-3.14159 upper=3.14159 effort=0.0 velocity=0.0
- added joint 6_7: type revolute, parent 6, child 7, origin xyz=0.8098941087802216 0 0 rpy=0 0 0, axis 0 0 1, limit lower=-3.14159 upper=3.14159 effort=0.0 velocity=0.0
